File: Encoder Board/Encoder Board.kicad_pcb (KiCad board)
At the start: 2 copper layers, 48 x 54 mm, 18 parts, among them J1 Conn_02x05_Odd_Even, J2 Conn_02x05_Odd_Even, J3 Conn_01x01_Pin, J4 Conn_01x01_Pin, U1 AM26LV32xD

Commit message: Add descriptive labels to silkscreen
Parts:
- J3, J4: value Conn_01x01_Pin -> Conn_01x02_Pin; footprint Connector_PinHeader_2.54mm:PinHeader_1x01_P2.54mm_Vertical -> Connector_PinHeader_2.54mm:PinHeader_1x02_P2.54mm_Vertical
- moved J3 29.8 mm to (122.5, 59.2)
- moved J4 26.2 mm to (122.5, 86.2)
- moved GND_1 9.06 mm to (90.0, 76.0)
Connections:
- J3 pad 1: /TRIGGER -> +5V_S
- J4 pad 1: +5V_S -> /TRIGGER
Routing:
- net /TRIGGER: track 17.3 -> 14.6 mm
- net +5V_S: track 11.8 -> 11.1 mm
Other:
- board text added: "ENCODER IN"
- board text added: "Encoder Trigger Board Rev. 1 Kailash Rao"
- board text added: "MOTOR CONTROLLER OUT"
- board text added: "PWR"
- board text added: "TRIGGER"

Commit message: Fix J2 orientation
Parts:
- moved J2 10.4 mm to (120.7, 68.0), turned to 0 degrees
- moved GND_1 1.80 mm to (91.5, 77.0)
Routing:
- net /B: track 62.6 -> 71.8 mm, vias 0 -> 1
- net GND: track 5.80 -> 14.9 mm, vias 3 -> 5
- net /INDEX_N: track 67.9 -> 63.1 mm, vias 0 -> 2
- net +5V_E: track 43.5 -> 47.9 mm, vias 0 -> 2
- net /INDEX: track 77.5 -> 81.1 mm, vias 0 -> 2
- net /A: track 71.5 -> 74.9 mm
- net /A_N: track 87.0 -> 84.5 mm
- net /B_N: track 58.4 -> 60.9 mm, vias 0 -> 1
