File: Encoder Board/Encoder Board.kicad_sch (KiCad schematic)
At the start: 24 parts, among them J1 Conn_02x05_Odd_Even, J2 Conn_02x05_Odd_Even, J3 Conn_01x02_Pin, J4 Conn_01x02_Pin, J4x1 Conn_01x02_Pin, J5 Conn_01x20, J6 Conn_01x20, J7 Conn_02x04_Odd_Even, U1 AM26LV32xD

Commit message: fix J1/J2 footprint
Parts:
- J1, J2: footprint Connector_PinHeader_2.54mm:PinHeader_2x05_P2.54mm_Vertical -> Clip Connector Library:PinSocket_2x05_P2.54mm_Vertical_ClipConnector
Changed lines of the file:
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@@
 			)
 		)
-		(property "Footprint" "Connector_PinHeader_2.54mm:PinHeader_2x05_P2.54mm_Vertical"
+		(property "Footprint" "Clip Connector Library:PinSocket_2x05_P2.54mm_Vertical_ClipConnector"
 			(at 34.29 31.75 0)
 			(hide yes)
@@
 			)
 		)
-		(property "Footprint" "Connector_PinHeader_2.54mm:PinHeader_2x05_P2.54mm_Vertical"
+		(property "Footprint" "Clip Connector Library:PinSocket_2x05_P2.54mm_Vertical_ClipConnector"
 			(at 259.08 30.48 0)
 			(hide yes)

Commit message: routing
Connections:
- net B: now also R3.2, U1.10 (3A); no longer R2.2, U1.6 (2A)
- net B_3V3: now also J5.6 (Pin_6), U1.11 (3Y); no longer J5.5 (Pin_5), U1.5 (2Y)
- net B_N: now also C3.1, U1.9 (3B); no longer C2.1, U1.7 (2B)
- net INDEX: now also R2.2, U1.6 (2A); no longer R3.2, U1.10 (3A)
- net INDEX_3V3: now also J5.5 (Pin_5), U1.5 (2Y); no longer J5.6 (Pin_6), U1.11 (3Y)
- net INDEX_N: now also C2.1, U1.7 (2B); no longer C3.1, U1.9 (3B)
Changed lines of the file:
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@@
+	(wire
+		(pts
+			(xy 73.66 38.1) (xy 111.76 38.1)
+		)
+		(stroke
+			(width 0)
+			(type default)
+		)
+	)
 	(wire
 		(pts
@@
 		(pts
 			(xy 254 16.51) (xy 260.35 16.51)
-		)
-		(stroke
-			(width 0)
-			(type default)
-		)
-	)
-	(wire
-		(pts
-			(xy 73.66 38.1) (xy 111.76 38.1)
 		)
 		(stroke
@@
 	)
 	(label "B_N"
-		(at 96.52 43.18 180)
+		(at 96.52 63.5 180)
 		(effects
 			(font
@@
 		)
 	)
+	(label "B_3V3"
+		(at 33.02 134.62 180)
+		(effects
+			(font
+				(size 1.27 1.27)
+			)
+			(justify right bottom)
+		)
+	)
 	(label "INDEX_3V3"
-		(at 142.24 60.96 0)
+		(at 142.24 40.64 0)
 		(effects
 			(font
@@
 	)
 	(label "B"
-		(at 93.98 38.1 180)
+		(at 93.98 58.42 180)
 		(effects
 			(font
@@
 	)
 	(label "INDEX_N"
-		(at 101.6 63.5 180)
+		(at 99.06 43.18 180)
 		(effects
 			(font
@@
 		)
 	)
+	(label "INDEX_3V3"
+		(at 33.02 132.08 180)
+		(effects
+			(font
+				(size 1.27 1.27)
+			)
+			(justify right bottom)
+		)
+	)
 	(label "B_3V3"
-		(at 142.24 40.64 0)
+		(at 142.24 60.96 0)
 		(effects
 			(font
@@
 		)
 	)
-	(label "B_3V3"
-		(at 33.02 132.08 180)
-		(effects
-			(font
-				(size 1.27 1.27)
-			)
-			(justify right bottom)
-		)
-	)
-	(label "INDEX_3V3"
-		(at 33.02 134.62 180)
-		(effects
-			(font
-				(size 1.27 1.27)
-			)
-			(justify right bottom)
-		)
-	)
 	(label "A_N"
 		(at 29.21 31.75 180)
@@
 	)
 	(label "INDEX"
-		(at 99.06 58.42 180)
-		(effects
-			(font
+		(at 96.52 38.1 180)
+		(effects
+			(font
