File: Encoder Board/_restore_backup_2026-05-30T00-43-04-764/Encoder Board.kicad_sch (KiCad schematic)
At the start: 24 parts, among them J1 Conn_02x05_Odd_Even, J2 Conn_02x05_Odd_Even, J3 Conn_01x02_Pin, J4 Conn_01x02_Pin, J4x1 Conn_01x02_Pin, J5 Conn_01x20, J6 Conn_01x20, J7 Conn_02x04_Odd_Even, U1 AM26LV32xD

Commit message: add BWRC logo, generate new gerbers
Parts:
- removed J7: Conn_02x04_Odd_Even, Connector_PinHeader_2.54mm:PinHeader_2x04_P2.54mm_Vertical, symbol Connector_Generic:Conn_02x04_Odd_Even
- added J7: Conn_02x04_Counter_Clockwise, Connector_PinHeader_2.54mm:PinHeader_2x04_P2.54mm_Vertical, symbol Connector_Generic:Conn_02x04_Counter_Clockwise
Connections:
- net GND: now also J7.5 (Pin_5), J7.6 (Pin_6), J7.7 (Pin_7), J7.8 (Pin_8)
- net TRIGGER: now also J7.1 (Pin_1)
- net at J6.15 (Pin_15): now also J7.2 (Pin_2)
- net at J6.16 (Pin_16): now also J7.3 (Pin_3)
- net at J6.17 (Pin_17): now also J7.4 (Pin_4)
