File: Encoder Board/_restore_backup_2026-06-01T11-58-52-217/Encoder Board.kicad_pcb (KiCad board)
At the start: 2 copper layers, 62.2 x 52.8 mm, 20 parts, among them J1 Conn_02x05_Odd_Even, J2 Conn_02x05_Odd_Even, J3 Conn_01x02_Pin, J4 Conn_01x02_Pin, J5 Conn_01x20, J6 Conn_01x20, J7 Conn_02x04_Odd_Even, U1 AM26LV32xD

Commit message: new placement
Routing:
- net /INDEX_3V3: track 5.75 -> 9.66 mm
- net /A_N: track 67.3 -> 69.6 mm
- net /INDEX: track 68.6 -> 70.5 mm
Changed lines of the file:
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@@
 				(font
 					(size 1.27 1.27)
-					(thickness 0.15)
 				)
 			)
@@
 				(font
 					(size 1.27 1.27)
-					(thickness 0.15)
 				)
 			)
@@
 				(font
 					(size 1.27 1.27)
-					(thickness 0.15)
 				)
 			)
@@
 				(font
 					(size 1.27 1.27)
-					(thickness 0.15)
 				)
 			)
@@
 				(font
 					(size 1.27 1.27)
-					(thickness 0.15)
 				)
 			)
@@
 				(font
 					(size 1.27 1.27)
-					(thickness 0.15)
 				)
 			)
@@
 				(font
 					(size 1.27 1.27)
-					(thickness 0.15)
 				)
 			)
@@
 				(font
 					(size 1.27 1.27)
-					(thickness 0.15)
 				)
 			)
@@
 				(font
 					(size 1.27 1.27)
-					(thickness 0.15)
 				)
 			)
@@
 				(font
 					(size 1.27 1.27)
-					(thickness 0.15)
 				)
 			)
@@
 				(font
 					(size 1.27 1.27)
-					(thickness 0.15)
 				)
 			)
@@
 				(font
 					(size 1.27 1.27)
-					(thickness 0.15)
 				)
 			)
@@
 				(font
 					(size 1.27 1.27)
-					(thickness 0.15)
 				)
 			)
@@
 				(font
 					(size 1.27 1.27)
-					(thickness 0.15)
 				)
 			)
@@
 				(font
 					(size 1.27 1.27)
-					(thickness 0.15)
 				)
 			)
@@
 				(font
 					(size 1.27 1.27)
-					(thickness 0.15)
 				)
 			)
@@
 				(font
 					(size 1.27 1.27)
-					(thickness 0.15)
 				)
 			)
@@
 	)
 	(via
-		(at 82.5 43.5)
+		(at 81.25 43)
 		(size 0.6)
 		(drill 0.3)
@@
 	)
 	(segment
+		(start 65.5745 49.267)
+		(end 67.1575 50.85)
+		(width 0.4)
+		(layer "F.Cu")
+		(net "/A_N")
+	)
+	(segment
 		(start 51.25 99.5)
 		(end 51.25 93.25)
@@
 	)
 	(segment
+		(start 76.668747 61.598747)
+		(end 75.32 60.25)
+		(width 0.4)
+		(layer "F.Cu")
+		(net "/INDEX")
+	)
+	(segment
 		(start 75.75 60.25)
 		(end 75.32 60.25)
@@
 	)
 	(segment
+		(start 81.738 44.306)
+		(end 84.5 47.068)
+		(width 0.4)
+		(layer "F.Cu")
+		(net "/INDEX_3V3")
+	)
+	(segment
 		(start 72.795 59.355)
 		(end 72.827 59.323)
@@
 		(polygon
 			(pts
-				(xy 81.393586 39.210744) (xy 81.406422 58.400105) (xy 65.857174 58.399956) (xy 65.902103 47.573863)
-				(xy 77.396786 47.621576) (xy 77.461881 31.032168) (xy 116.994215 31.187296) (xy 117.008019 58.777208)
+				(xy 82.393585 39.21013) (xy 82.40642 58.400044) (xy 65.857174 58.399956) (xy 65.902103 47.573863)
+				(xy 78.396758 47.625718) (xy 78.461853 31.0361) (xy 116.994215 31.187296) (xy 117.008019 58.777208)
 				(xy 112.009037 58.778788) (xy 111.99368 39.189878)
 			)
